Commit message: simulation works good

File: articubot_one/description/depth_camera.xacro (robot description, xacro)
@@ -1,30 +1,76 @@
 <?xml version="1.0"?>
 <robot xmlns:xacro="http://www.ros.org/wiki/xacro" >
-    <joint name="camera_joint" type="fixed">
+<!-- FRONT DEPTH CAMERA  -->
+    <joint name="front_depth_camera_joint" type="fixed">
         <parent link="chassis"/>
-        <child link="camera_link"/>
-        <origin xyz="0.305 0 0.08" rpy="0 0 0"/>
+        <child link="front_depth_camera"/>
+        <origin xyz="0.625 0 0.43" rpy="0 0.96 0"/>
     </joint>
-    <link name="camera_link">
+    <link name="front_depth_camera">
         <visual>
             <geometry>
-                <box size="0.010 0.03 0.03"/>
+                <box size="0.010 0.06 0.03"/>
             </geometry>
             <material name="red"/>
         </visual>
     </link>
-    <joint name="camera_optical_joint" type="fixed">
-        <parent link="camera_link"/>
-        <child link="camera_link_optical"/>
+    <joint name="front_depth_camera_optical_joint" type="fixed">
+        <parent link="front_depth_camera"/>
+        <child link="front_depth_camera_optical"/>
         <origin xyz="0 0 0" rpy="${-pi/2} 0 ${-pi/2}"/>
     </joint>
-    <link name="camera_link_optical"></link>
-    <gazebo reference="camera_link">
+    <link name="front_depth_camera_optical"></link>
+    <gazebo reference="front_depth_camera">
         <material>Gazebo/Red</material>
-        <sensor name="camera" type="depth">
+        <sensor name="front_depth_camera" type="depth">
             <pose> 0 0 0 0 0 0 </pose>
             <visualize>true</visualize>
             <update_rate>10</update_rate>
-            <camera>
+            <front_depth_camera>
+                <horizontal_fov>0.8</horizontal_fov>
+                <image>
+                    <format>B8G8R8</format>
+                    <width>640</width>
+                    <height>480</height>
+                </image>
+                <clip>
+                    <near>0.05</near>
+                    <far>8.0</far>
+                </clip>
+            </front_depth_camera>
+            <plugin name="front_depth_camera_controller" filename="libgazebo_ros_camera.so">
+                <frame_name>front_depth_camera_optical</frame_name>
+                <min_depth>0.1</min_depth>
+                <max_depth>100.0</max_depth>
+            </plugin>
+        </sensor>
+    </gazebo>
+<!-- REAR DEPTH CAMERA  -->
+    <joint name="rear_depth_camera_joint" type="fixed">
+        <parent link="chassis"/>
+        <child link="rear_depth_camera"/>
+        <origin xyz="-0.645 0 0.43" rpy="0 0.4 ${pi}"/>
+    </joint>
+    <link name="rear_depth_camera">
+        <visual>
+            <geometry>
+                <box size="0.010 0.06 0.03"/>
+            </geometry>
+            <material name="red"/>
+        </visual>
+    </link>
+    <joint name="rear_depth_camera_optical_joint" type="fixed">
+        <parent link="rear_depth_camera"/>
+        <child link="rear_depth_camera_optical"/>
+        <origin xyz="0 0 0" rpy="${-pi/2} 0 ${-pi/2}"/>
+    </joint>
+    <link name="rear_depth_camera_optical"></link>
+    <gazebo reference="rear_depth_camera">
+        <material>Gazebo/Red</material>
+        <sensor name="rear_depth_camera" type="depth">
+            <pose> 0 0 0 0 0 0 </pose>
+            <visualize>true</visualize>
+            <update_rate>10</update_rate>
+            <rear_depth_camera>
                 <horizontal_fov>1.089</horizontal_fov>
                 <image>
@@ -37,7 +83,7 @@
                     <far>8.0</far>
                 </clip>
-            </camera>
-            <plugin name="camera_controller" filename="libgazebo_ros_camera.so">
-                <frame_name>camera_link_optical</frame_name>
+            </rear_depth_camera>
+            <plugin name="rear_depth_camera_controller" filename="libgazebo_ros_camera.so">
+                <frame_name>rear_depth_camera_optical</frame_name>
                 <min_depth>0.1</min_depth>
                 <max_depth>100.0</max_depth>

File: articubot_one/description/robot.urdf.xacro (robot description, xacro)
@@ -11,7 +11,6 @@
     </xacro:unless>
     <xacro:include filename="lidar.xacro" />
-    <xacro:include filename="camera.xacro" />
+    <!-- <xacro:include filename="camera.xacro" /> -->
     <xacro:include filename="imu.xacro" />
-    <!-- <xacro:include filename="depth_camera.xacro" /> -->
-    <xacro:include filename="face.xacro" />
+    <xacro:include filename="depth_camera.xacro" />
 </robot>

File: articubot_one/description/robot_core.xacro (robot description, xacro)
@@ -4,5 +4,5 @@
     <xacro:property name="chassis_length" value="1.2"/>
     <xacro:property name="chassis_width" value="1.0"/>
-    <xacro:property name="chassis_height" value="0.17"/>
+    <xacro:property name="chassis_height" value="0.01"/>
     <xacro:property name="chassis_mass" value="10.0"/>
     <xacro:property name="wheel_radius" value="0.2"/>
@@ -10,7 +10,7 @@
     <xacro:property name="wheel_mass" value="1.0"/>
     <xacro:property name="wheel_offset_x" value="0.10"/>
-    <xacro:property name="wheel_offset_y" value="0.55"/>
+    <xacro:property name="wheel_offset_y" value="0.535"/>
     <xacro:property name="wheel_offset_z" value="-0.050"/>
-    <xacro:property name="wheel_seperate_x" value="0.35"/>
+    <xacro:property name="wheel_seperate_x" value="0.325"/>
     <xacro:property name="caster_wheel_radius" value="0.0175"/>
     <xacro:property name="caster_wheel_mass" value="0.1"/>
@@ -51,7 +51,7 @@
     <link name="chassis">
         <visual>
-            <origin xyz="-0.613255 -0.702 -0.15" rpy="0 0 0" />
-            <geometry>
-                <mesh filename="$(find articubot_one)/description/mesh/body2.STL"/>$
+            <origin xyz="0 0 -0.075" rpy="0 0 0" />
+            <geometry>
+                <mesh filename="$(find articubot_one)/description/mesh/blender_top.stl"/>$
             </geometry>
             <material name="orange"/>
@@ -75,14 +75,21 @@
         <parent link="base_link"/>
         <child link="chassis_top"/>
-        <origin xyz="0 0 0" rpy="0 0 0" />
+        <origin xyz="0 0 0"/>
     </joint>
     <link name="chassis_top">
         <visual>
-            <origin xyz="-0.555323 -0.623625 -0.15" rpy="0 0 0"/>
-            <geometry>
-                <mesh filename="$(find articubot_one)/description/mesh/body1.STL"/>$
+            <origin xyz="0 0 -0.075" rpy="0 0 0" />
+            <geometry>
+                <mesh filename="$(find articubot_one)/description/mesh/blender_body.stl"/>$
             </geometry>
             <material name="red"/>
         </visual>
+        <collision>
+            <origin xyz="0 0 0"/>
+            <geometry>
+                <box size="1.0 0.5 0.1"/>
+            </geometry>
+            <material name="red"/>
+        </collision>
         <xacro:inertial_box mass="0.5" x="${chassis_length}" y="${chassis_width}" z="${chassis_height}">
             <origin xyz="0 0 0" rpy="0 0 0"/>
@@ -90,5 +97,5 @@
     </link>
     <gazebo reference="chassis_top">
-        <material>Gazebo/red</material>
+        <material>Gazebo/Red</material>
     </gazebo>
     <!-- FRONT LEFT WHEEL LINK -->
@@ -102,6 +109,7 @@
     <link name="front_left_wheel">
         <visual>
-            <geometry>
-                <cylinder radius="${wheel_radius}" length="${wheel_thickness}"/>
+            <origin xyz="0 0 0" rpy="0 ${pi} 0" />
+            <geometry>
+                <mesh filename="$(find articubot_one)/description/mesh/blender_wheel.stl"/>$
             </geometry>
             <material name="blue"/>
@@ -131,6 +139,7 @@
     <link name="rear_left_wheel">
         <visual>
-            <geometry>
-                <cylinder radius="${wheel_radius}" length="${wheel_thickness}"/>
+            <origin xyz="0 0 0" rpy="0 ${pi} 0" />
+            <geometry>
+                <mesh filename="$(find articubot_one)/description/mesh/blender_wheel.stl"/>$
             </geometry>
             <material name="blue"/>
@@ -160,6 +169,7 @@
     <link name="front_right_wheel">
         <visual>
-            <geometry>
-                <cylinder radius="${wheel_radius}" length="${wheel_thickness}"/>
+            <origin xyz="0 0 0" rpy="0 ${pi} 0" />
+            <geometry>
+                <mesh filename="$(find articubot_one)/description/mesh/blender_wheel.stl"/>$
             </geometry>
             <material name="blue"/>
@@ -189,6 +199,7 @@
     <link name="rear_right_wheel">
         <visual>
-            <geometry>
-                <cylinder radius="${wheel_radius}" length="${wheel_thickness}"/>
+            <origin xyz="0 0 0" rpy="0 ${pi} 0" />
+            <geometry>
+                <mesh filename="$(find articubot_one)/description/mesh/blender_wheel.stl"/>$
             </geometry>
             <material name="blue"/>
